File: PumpMonitor/PumpMonitorVeroboardLayout/PumpMonitor.kicad_pcb (KiCad board)
At the start: 2 copper layers, 119.4 x 55.9 mm, 29 parts, among them J1 Power & Current Sense, J2 Programming, J3 Ra01_Breakout_Module, Q1 BC548, Q2 BC548, SW1 SW_Push, U1 LM317_TO-220, U2 24LC16, U3 PICAXE-18M2

Commit message: Cleaning up and adding resetting + temperature consisency detection
Connections:
- U2 pad 1: Net-(U2-Pad1) -> unconnected-(U2-Pad1)
- U2 pad 2: Net-(U2-Pad2) -> unconnected-(U2-Pad2)
- U2 pad 3: Net-(U2-Pad3) -> unconnected-(U2-Pad3)
- U2 pad 7: Net-(U2-Pad7) -> unconnected-(U2-Pad7)
- U3 pad 11: Net-(U3-Pad11) -> unconnected-(U3-Pad11)
- U3 pad 8: Net-(U3-Pad8) -> unconnected-(U3-Pad8)
Other:
- net class Default removed
