File: IrrigationWaterDetector/WaterbabyLayout/WaterbabyLayout.kicad_sch (KiCad schematic)
At the start: 15 parts, among them J1 Power, J2 Programming, J3 Sensor, U1 Ra01_Breakout_Module, U2 PICAXE-14M2

Commit message: Started gate monitor, fence monitor code adapted mostly
Other:
- title: Electric fence monitor -> Water baby
Changed lines of the file:
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@@
 	(paper "A4")
 	(title_block
-		(title "Electric fence monitor")
+		(title "Water baby")
 		(date "2024-11-09")
 		(company "Jotham Gates")
